File: build/mysTeleinfo.sch (KiCad schematic (older format))
At the start: 14 parts, among them P1 CNX2, P2 CNX2, P9 CONN_01X06, Q1 BS170, U1 ArduinoNano, U2 NRF24L01, U3 LTV-814

Commit message: mysTeleinfo: prepare 3.0 - use Linky TIC standard
Parts:
- removed P1, P2: CNX2, symbol CONN_01X02
- removed P9: CONN_01X06, symbol CONN_01X06
- removed Q1: BS170, TO-92, symbol BS170
- removed R1, R5, R6, R7: 220, symbol R
- removed R2: 4,7k, symbol R
- removed R3, R4: 10k, symbol R
- removed U3: LTV-814, DIP-4, symbol LTV-814
- added P1: Power, symbol Connector:Screw_Terminal_01x02
- added P2: Téléinfo, symbol Connector:Screw_Terminal_01x02
- added P9: LED Panel, symbol Connector:Screw_Terminal_01x05
- added R1: 1,2k, symbol Device:R
- added R2*: 4,7k, symbol Device:R
- added R3, R4, R5, R6: 220, symbol Device:R
- added U3: LTV-814A, DIP-4, symbol Isolator:LTV-824
- U1: symbol ArduinoNano -> arduinonano:ArduinoNano
- U2: symbol NRF24L01 -> arduinonano:NRF24L01
Connections:
- net +5V: now also P1.1 (Pin_1), R2*.2, R6.2
- net GND: now also P1.2 (Pin_2), P9.5 (Pin_5), U3.7
- net at U1.10 (D7): now also R3.2
- net at U1.7 (D4): now also R2*.1, U3.8
- net at U1.8 (D5): now also R5.2
- net at U1.9 (D6): now also R4.2
- new net: P2.1 (Pin_1), R1.1
- new net: P2.2 (Pin_2), U3.1
- new net: P9.1 (Pin_1), R6.1
- new net: P9.2 (Pin_2), R5.1
- new net: P9.3 (Pin_3), R4.1
- new net: P9.4 (Pin_4), R3.1
- new net: R1.2, U3.2
Other:
- note added: "- +5v (green)\n- Teleinfo (green)\n- HC LED (yellow)\n- HP LED (orange)\n- GND"
- note added: "Source : https://imagesia.com/intteleinfo007_8g2"
- note removed: "D4"
- note removed: "LED Panel\n- Teleinfo (green)\n- +5v (green)\n- HC LED (yellow)\n- HP LED (orange)\n\n- GND"
- note removed: "Téléinfo"
- moved on the sheet: U2
